Commit message: Refactor xarm6 URDF: removed unused materials and links, added force torque sensor and camera stand links with fixed joints, and updated joint configurations for improved functionality.

File: xarm6_with_gripper_v1.urdf (robot description, URDF)
Before this commit: robot xarm6_with_gripper_v1, 16 links, 15 joints
Links:
- added link link_camera_stand, mass 0.1; collision mesh filename=collision/cam_stand.stl; visual mesh filename=collision/cam_stand.stl
- added link link_ft_sensor, mass 0.3; collision mesh filename=collision/ft_sensor.stl scale=0.001 0.001 0.001; visual mesh filename=collision/ft_sensor.stl scale=0.001 0.001 0.001
Joints:
- added joint joint_sensor_fix: type fixed, parent link6, child link_ft_sensor, origin xyz=-0.0375 -0.0375 0.006 rpy=0 0 0
- added joint joint_stand_fix: type fixed, parent link_ft_sensor, child link_camera_stand, origin xyz=0.0375 0.0375 0.055 rpy=0 0 0
- joint gripper_base_joint: origin xyz=0 0 0 rpy=0 0 0 -> xyz=0 0 0.005 rpy=0 0 0; parent link6 -> link_camera_stand
- joint joint_tcp: origin xyz=0 0 0 rpy=0 0 0 -> xyz=0 0 -0.005 rpy=0 0 0
- joint left_finger_joint: axis 1 0 0 -> -1 0 0; limit lower=-0.85 upper=0 effort=50 velocity=2.0 -> lower=0 upper=0.85 effort=50 velocity=2.0; mimic (none) -> joint=drive_joint multiplier=1 offset=0
- joint left_inner_knuckle_joint: mimic (none) -> joint=drive_joint multiplier=1 offset=0
- joint right_finger_joint: mimic (none) -> joint=drive_joint multiplier=1 offset=0
- joint right_inner_knuckle_joint: mimic (none) -> joint=drive_joint multiplier=1 offset=0
- joint right_outer_knuckle_joint: mimic (none) -> joint=drive_joint multiplier=1 offset=0

Commit message: Remove unused FT sensor link and joint from xarm6 URDF; update joint parent link for camera stand to improve model structure.

File: xarm6_with_gripper_v1.urdf (robot description, URDF)
Before this commit: robot xarm6_with_gripper_v1, 18 links, 17 joints
Links:
- removed link link_ft_sensor
Joints:
- removed joint joint_sensor_fix
- joint joint_stand_fix: origin xyz=0.0375 0.0375 0.055 rpy=0 0 0 -> xyz=0 0 0 rpy=0 0 0; parent link_ft_sensor -> link6
